File: Schematic/Apple2c VGA kicad/apple2c VGA/apple2c VGA.kicad_pcb (KiCad board)
At the start: 2 copper layers, 53.3 x 48.3 mm, 32 parts, among them J1 DB15_Male, J2 DB15_Female_HighDensity, J3 Conn_01x14_Female, J4 Conn_01x14_Female, Q1 BSS138, Q2 BSS138, Q3 BSS138, Q4 BSS138, SW1 SW_Push_Dual, U1 MIC5205-5.0YM5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

Commit message: Tidy up
Other:
- board text added: "Apple2c VGA v2.0"
